File: CNC-MainStepInterface-panel.sch (EAGLE design)
At the start: 30 parts, among them IC10 ATTINY84-20PU, IC11 74HCT595N, IC1A ARDUINO_MINI, IC1B ATMEGA328P_PDIP, IC2 74HCT541N, IC3 74HCT541N, IC4 74HCT541N, IC5 74HCT541N, IC6 ATTINY2313A-PU, IC7 74HCT125N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

Commit message: BUGFIX: [XYZ]_LIMIT# not connected to [XYZ]_HOME# - when panelizing Main + Stepper + Interface on the same board, I forgot to make LIMIT the same as HOME. This will have to be reworked by hand during assembly. - only added net connections, PCB artwork to be updated at the next autorouter run - added 45 degree corners to some traces that escaped the first pass
Connections:
- removed net !X_LIMIT: IC8.(PCINT10/INT0/OC0A/CKOUT)PB2
- removed net !Y_LIMIT: IC9.(PCINT10/INT0/OC0A/CKOUT)PB2
- removed net !Z_LIMIT: IC10.(PCINT10/INT0/OC0A/CKOUT)PB2
- net !X_HOME: now also IC8.(PCINT10/INT0/OC0A/CKOUT)PB2
- net !Y_HOME: now also IC9.(PCINT10/INT0/OC0A/CKOUT)PB2
- net !Z_HOME: now also IC10.(PCINT10/INT0/OC0A/CKOUT)PB2
Changed lines of the file:
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@@
 <label x="124.46" y="96.52" size="1.778" layer="95" rot="R90"/>
+</segment>
+<segment>
+<pinref part="IC8" gate="G$1" pin="(PCINT10/INT0/OC0A/CKOUT)PB2"/>
+<wire x1="396.24" y1="139.7" x2="419.1" y2="139.7" width="0.1524" layer="91"/>
+<label x="411.48" y="139.7" size="1.778" layer="95"/>
 </segment>
 </net>
@@
 <label x="127" y="96.52" size="1.778" layer="95" rot="R90"/>
 </segment>
+<segment>
+<pinref part="IC9" gate="G$1" pin="(PCINT10/INT0/OC0A/CKOUT)PB2"/>
+<wire x1="396.24" y1="96.52" x2="419.1" y2="96.52" width="0.1524" layer="91"/>
+<label x="411.48" y="96.52" size="1.778" layer="95"/>
+</segment>
 </net>
 <net name="!Z_HOME" class="0">
@@
 <wire x1="129.54" y1="157.48" x2="129.54" y2="96.52" width="0.1524" layer="91"/>
 <label x="129.54" y="96.52" size="1.778" layer="95" rot="R90"/>
+</segment>
+<segment>
+<pinref part="IC10" gate="G$1" pin="(PCINT10/INT0/OC0A/CKOUT)PB2"/>
+<wire x1="396.24" y1="53.34" x2="419.1" y2="53.34" width="0.1524" layer="91"/>
+<label x="411.48" y="53.34" size="1.778" layer="95"/>
 </segment>
 </net>
@@
 </segment>
 </net>
-<net name="!X_LIMIT" class="0">
-<segment>
-<pinref part="IC8" gate="G$1" pin="(PCINT10/INT0/OC0A/CKOUT)PB2"/>
-<wire x1="396.24" y1="139.7" x2="419.1" y2="139.7" width="0.1524" layer="91"/>
-<label x="411.48" y="139.7" size="1.778" layer="95"/>
-</segment>
-</net>
-<net name="!Y_LIMIT" class="0">
-<segment>
-<pinref part="IC9" gate="G$1" pin="(PCINT10/INT0/OC0A/CKOUT)PB2"/>
-<wire x1="396.24" y1="96.52" x2="419.1" y2="96.52" width="0.1524" layer="91"/>
-<label x="411.48" y="96.52" size="1.778" layer="95"/>
-</segment>
-</net>
-<net name="!Z_LIMIT" class="0">
-<segment>
-<pinref part="IC10" gate="G$1" pin="(PCINT10/INT0/OC0A/CKOUT)PB2"/>
-<wire x1="396.24" y1="53.34" x2="419.1" y2="53.34" width="0.1524" layer="91"/>
-<label x="411.48" y="53.34" size="1.778" layer="95"/>
-</segment>
-</net>
